Commit message: Add eye geometry and URDF updates

File: urdf/ee/openarm_hand.xacro (robot description, xacro)
@@ -24,4 +24,11 @@
       <parent link="${ee_prefix}hand" />
       <child link="${ee_prefix}hand_tcp" />
+    </joint>
+    <!-- Planning tip frame, available in both fake and real hardware chains -->
+    <link name="${ee_prefix}gripper_tip" />
+    <joint name="${ee_prefix}gripper_tip_joint" type="fixed">
+      <origin xyz="0 0 0" rpy="0 0 0" />
+      <parent link="${ee_prefix}hand_tcp" />
+      <child link="${ee_prefix}gripper_tip" />
     </joint>
     <link name="${ee_prefix}left_finger">

File: urdf/robot/v10.urdf.xacro (robot description, xacro)
@@ -2,4 +2,5 @@
 <robot xmlns:xacro="http://www.ros.org/wiki/xacro" name="openarm">
   <xacro:include filename="$(find openarm_description)/urdf/robot/openarm_robot.xacro"/>
+  <xacro:include filename="$(find openarm_description)/urdf/eye/_d435.urdf.xacro"/>
   <xacro:arg name="arm_type" default="v10" />
   <xacro:arg name="body_type" default="v10" />
@@ -27,4 +28,5 @@
   <xacro:arg name="left_arm_base_rpy" default="-1.5708 0 0" />
   <xacro:arg name="can_fd" default="true" />
+  <xacro:arg name="enable_d435" default="true" />
   <xacro:openarm_robot
   arm_type="v10"
@@ -62,3 +64,8 @@
   can_fd="$(arg can_fd)"
   />
+  <!-- <xacro:if value="$(arg enable_d435)">
+    <xacro:sensor_d435 parent="world" name="camera1" use_nominal_extrinsics="true">
+      <origin xyz="0.32034904 0.05333502 0.73377816" rpy=" 3.1376668 -0.0537802 -1.5810559"/>
+    </xacro:sensor_d435>
+  </xacro:if> -->
 </robot>
